File: blackbox-ng/MPU9250.sch (KiCad schematic (older format))
At the start: 4 parts

Commit message: assign footprints
Parts:
- C19, C20, C21: renamed from C?; footprint (none) -> Capacitor_SMD:C_0603_1608Metric_Pad1.05x0.95mm_HandSolder
- gave numbers to parts that had none: 1
Changed lines of the file:
@@
 $EndDescr
 $Comp
-L Sensor_Motion:MPU-9250 U?
+L Sensor_Motion:MPU-9250 U4
 U 1 1 5DF48C70
 P 5900 3250
-F 0 "U?" H 5900 2261 50  0000 C CNN
+F 0 "U4" H 5900 2261 50  0000 C CNN
 F 1 "MPU-9250" H 5900 2170 50  0000 C CNN
 F 2 "Sensor_Motion:InvenSense_QFN-24_3x3mm_P0.4mm" H 5900 2250 50  0001 C CNN
@@
 $EndComp
 $Comp
-L power:VDD #PWR?
+L power:VDD #PWR0132
 U 1 1 5DF49450
 P 5800 2150
-F 0 "#PWR?" H 5800 2000 50  0001 C CNN
+F 0 "#PWR0132" H 5800 2000 50  0001 C CNN
 F 1 "VDD" H 5817 2323 50  0000 C CNN
 F 2 "" H 5800 2150 50  0001 C CNN
@@
 Connection ~ 5800 2350
 $Comp
-L power:VDD #PWR?
+L power:VDD #PWR0133
 U 1 1 5DF498F3
 P 7100 3550
-F 0 "#PWR?" H 7100 3400 50  0001 C CNN
+F 0 "#PWR0133" H 7100 3400 50  0001 C CNN
 F 1 "VDD" H 7117 3723 50  0000 C CNN
 F 2 "" H 7100 3550 50  0001 C CNN
@@
 $EndComp
 $Comp
-L power:GND #PWR?
+L power:GND #PWR0134
 U 1 1 5DF49B99
 P 7100 3650
-F 0 "#PWR?" H 7100 3400 50  0001 C CNN
+F 0 "#PWR0134" H 7100 3400 50  0001 C CNN
 F 1 "GND" H 7105 3477 50  0000 C CNN
 F 2 "" H 7100 3650 50  0001 C CNN
@@
 	7100 3550 6600 3550
 $Comp
-L Device:C_Small C?
+L Device:C_Small C21
 U 1 1 5DF49EA4
 P 7450 3600
-F 0 "C?" H 7542 3646 50  0000 L CNN
+F 0 "C21" H 7542 3646 50  0000 L CNN
 F 1 "100n" H 7542 3555 50  0000 L CNN
-F 2 "" H 7450 3600 50  0001 C CNN
+F 2 "Capacitor_SMD:C_0603_1608Metric_Pad1.05x0.95mm_HandSolder" H 7450 3600 50  0001 C CNN
 F 3 "~" H 7450 3600 50  0001 C CNN
 	1    7450 3600
@@
 Connection ~ 7100 3650
 $Comp
-L Device:C_Small C?
+L Device:C_Small C20
 U 1 1 5DF4A514
 P 7100 3200
-F 0 "C?" V 6871 3200 50  0000 C CNN
+F 0 "C20" V 6871 3200 50  0000 C CNN
 F 1 "100n" V 6962 3200 50  0000 C CNN
-F 2 "" H 7100 3200 50  0001 C CNN
+F 2 "Capacitor_SMD:C_0603_1608Metric_Pad1.05x0.95mm_HandSolder" H 7100 3200 50  0001 C CNN
 F 3 "~" H 7100 3200 50  0001 C CNN
 	1    7100 3200
@@
 	6900 3200 7000 3200
 $Comp
-L power:GND #PWR?
+L power:GND #PWR0135
 U 1 1 5DF4BDD8
 P 7400 3200
-F 0 "#PWR?" H 7400 2950 50  0001 C CNN
+F 0 "#PWR0135" H 7400 2950 50  0001 C CNN
 F 1 "GND" H 7405 3027 50  0000 C CNN
 F 2 "" H 7400 3200 50  0001 C CNN
@@
 NoConn ~ 6600 3250
 $Comp
-L power:GND #PWR?
+L power:GND #PWR0136
 U 1 1 5DF4C5DB
 P 5900 4450
-F 0 "#PWR?" H 5900 4200 50  0001 C CNN
+F 0 "#PWR0136" H 5900 4200 50  0001 C CNN
 F 1 "GND" H 5905 4277 50  0000 C CNN
 F 2 "" H 5900 4450 50  0001 C CNN
@@
 	5200 2950 5050 2950
 $Comp
-L power:VDD #PWR?
+L power:VDD #PWR0137
 U 1 1 5DF4D597
 P 4900 3450
-F 0 "#PWR?" H 4900 3300 50  0001 C CNN
+F 0 "#PWR0137" H 4900 3300 50  0001 C CNN
 F 1 "VDD" H 4917 3623 50  0000 C CNN
 F 2 "" H 4900 3450 50  0001 C CNN
@@
 NoConn ~ 5200 3450
 $Comp
-L Device:C_Small C?
+L Device:C_Small C19
 U 1 1 5DF4EF83
 P 6100 2250
-F 0 "C?" V 5871 2250 50  0000 C CNN
+F 0 "C19" V 5871 2250 50  0000 C CNN
 F 1 "10n" V 5962 2250 50  0000 C CNN
-F 2 "" H 6100 2250 50  0001 C CNN
+F 2 "Capacitor_SMD:C_0603_1608Metric_Pad1.05x0.95mm_HandSolder" H 6100 2250 50  0001 C CNN
 F 3 "~" H 6100 2250 50  0001 C CNN
 	1    6100 2250
@@
 $EndComp
 $Comp
-L power:GND #PWR?
+L power:GND #PWR0138
 U 1 1 5DF4F882
 P 6450 2300
-F 0 "#PWR?" H 6450 2050 50  0001 C CNN
+F 0 "#PWR0138" H 6450 2050 50  0001 C CNN
 F 1 "GND" H 6455 2127 50  0000 C CNN
 F 2 "" H 6450 2300 50  0001 C CNN
