File: blackbox-ng/STM32F401RET6.sch (KiCad schematic (older format))
At the start: 18 parts

Commit message: assign footprints
Parts:
- C10, C11, C12, C13, C14, C15, C3, C4, C5, C6, C7, C8, C9: renamed from C?; footprint (none) -> Capacitor_SMD:C_0603_1608Metric_Pad1.05x0.95mm_HandSolder
- FB1: renamed from FB?; footprint (none) -> Inductor_SMD:L_0603_1608Metric_Pad1.05x0.95mm_HandSolder
- R10, R11, R9: renamed from R?; footprint (none) -> Resistor_SMD:R_0603_1608Metric_Pad1.05x0.95mm_HandSolder
- gave numbers to parts that had none: 1
Changed lines of the file:
@@
 P 2800 4400
 AR Path="/5DDEFD3F" Ref="U?"  Part="1"
-AR Path="/5DDEE5E2/5DDEFD3F" Ref="U?"  Part="1"
-F 0 "U?" H 2750 6281 50  0000 C CNN
+AR Path="/5DDEE5E2/5DDEFD3F" Ref="U2"  Part="1"
+F 0 "U2" H 2750 6281 50  0000 C CNN
 F 1 "STM32F401RETx" H 2750 6190 50  0000 C CNN
 F 2 "Package_QFP:LQFP-64_10x10mm_P0.5mm" H 2200 2700 50  0001 R CNN
@@
 P 2550 2450
 AR Path="/5DDEFD4B" Ref="#PWR?"  Part="1"
-AR Path="/5DDEE5E2/5DDEFD4B" Ref="#PWR?"  Part="1"
-F 0 "#PWR?" H 2550 2300 50  0001 C CNN
+AR Path="/5DDEE5E2/5DDEFD4B" Ref="#PWR0120"  Part="1"
+F 0 "#PWR0120" H 2550 2300 50  0001 C CNN
 F 1 "VDD" H 2567 2623 50  0000 C CNN
 F 2 "" H 2550 2450 50  0001 C CNN
@@
 P 2050 2500
 AR Path="/5DDEFD5C" Ref="#PWR?"  Part="1"
-AR Path="/5DDEE5E2/5DDEFD5C" Ref="#PWR?"  Part="1"
-F 0 "#PWR?" H 2050 2250 50  0001 C CNN
+AR Path="/5DDEE5E2/5DDEFD5C" Ref="#PWR0121"  Part="1"
+F 0 "#PWR0121" H 2050 2250 50  0001 C CNN
 F 1 "GND" H 2055 2327 50  0000 C CNN
 F 2 "" H 2050 2500 50  0001 C CNN
@@
 P 2250 2450
 AR Path="/5DDEFD45" Ref="C?"  Part="1"
-AR Path="/5DDEE5E2/5DDEFD45" Ref="C?"  Part="1"
-F 0 "C?" V 2021 2450 50  0000 C CNN
+AR Path="/5DDEE5E2/5DDEFD45" Ref="C12"  Part="1"
+F 0 "C12" V 2021 2450 50  0000 C CNN
 F 1 "100n" V 2112 2450 50  0000 C CNN
-F 2 "" H 2250 2450 50  0001 C CNN
+F 2 "Capacitor_SMD:C_0603_1608Metric_Pad1.05x0.95mm_HandSolder" H 2250 2450 50  0001 C CNN
 F 3 "~" H 2250 2450 50  0001 C CNN
 	1    2250 2450
@@
 P 1300 2500
 AR Path="/5DE04F26" Ref="#PWR?"  Part="1"
-AR Path="/5DDEE5E2/5DE04F26" Ref="#PWR?"  Part="1"
-F 0 "#PWR?" H 1300 2250 50  0001 C CNN
+AR Path="/5DDEE5E2/5DE04F26" Ref="#PWR0122"  Part="1"
+F 0 "#PWR0122" H 1300 2250 50  0001 C CNN
 F 1 "GND" H 1305 2327 50  0000 C CNN
 F 2 "" H 1300 2500 50  0001 C CNN
@@
 P 1500 2450
 AR Path="/5DE04F2C" Ref="C?"  Part="1"
-AR Path="/5DDEE5E2/5DE04F2C" Ref="C?"  Part="1"
-F 0 "C?" V 1271 2450 50  0000 C CNN
+AR Path="/5DDEE5E2/5DE04F2C" Ref="C11"  Part="1"
+F 0 "C11" V 1271 2450 50  0000 C CNN
 F 1 "100n" V 1362 2450 50  0000 C CNN
-F 2 "" H 1500 2450 50  0001 C CNN
+F 2 "Capacitor_SMD:C_0603_1608Metric_Pad1.05x0.95mm_HandSolder" H 1500 2450 50  0001 C CNN
 F 3 "~" H 1500 2450 50  0001 C CNN
 	1    1500 2450
@@
 	1750 2450 1750 2900
 $Comp
-L Device:Ferrite_Bead_Small FB?
+L Device:Ferrite_Bead_Small FB1
 U 1 1 5DE0DDAE
 P 1700 3700
-F 0 "FB?" V 1463 3700 50  0000 C CNN
+F 0 "FB1" V 1463 3700 50  0000 C CNN
 F 1 "bead" V 1554 3700 50  0000 C CNN
-F 2 "" V 1630 3700 50  0001 C CNN
+F 2 "Inductor_SMD:L_0603_1608Metric_Pad1.05x0.95mm_HandSolder" V 1630 3700 50  0001 C CNN
 F 3 "~" H 1700 3700 50  0001 C CNN
 	1    1700 3700
@@
 	1800 3400 2100 3400
 $Comp
-L power:VDD #PWR?
+L power:VDD #PWR0123
 U 1 1 5DE0EC99
 P 1150 3700
-F 0 "#PWR?" H 1150 3550 50  0001 C CNN
+F 0 "#PWR0123" H 1150 3550 50  0001 C CNN
 F 1 "VDD" H 1167 3873 50  0000 C CNN
 F 2 "" H 1150 3700 50  0001 C CNN
@@
 	2100 4500 1900 4500
 $Comp
-L Device:C_Small C?
+L Device:C_Small C14
 U 1 1 5DE172A3
 P 1200 3300
-F 0 "C?" H 1108 3254 50  0000 R CNN
+F 0 "C14" H 1108 3254 50  0000 R CNN
 F 1 "100n" H 1108 3345 50  0000 R CNN
-F 2 "" H 1200 3300 50  0001 C CNN
+F 2 "Capacitor_SMD:C_0603_1608Metric_Pad1.05x0.95mm_HandSolder" H 1200 3300 50  0001 C CNN
 F 3 "~" H 1200 3300 50  0001 C CNN
 	1    1200 3300
@@
 $EndComp
 $Comp
-L Device:C_Small C?
+L Device:C_Small C15
 U 1 1 5DE1DB61
 P 1650 3300
-F 0 "C?" H 1742 3346 50  0000 L CNN
+F 0 "C15" H 1742 3346 50  0000 L CNN
 F 1 "1u" H 1742 3255 50  0000 L CNN
-F 2 "" H 1650 3300 50  0001 C CNN
+F 2 "Capacitor_SMD:C_0603_1608Metric_Pad1.05x0.95mm_HandSolder" H 1650 3300 50  0001 C CNN
 F 3 "~" H 1650 3300 50  0001 C CNN
 	1    1650 3300
@@
 	1200 3200 1650 3200
 $Comp
-L power:GND #PWR?
+L power:GND #PWR0124
 U 1 1 5DE1F48A
 P 1000 3200
-F 0 "#PWR?" H 1000 2950 50  0001 C CNN
+F 0 "#PWR0124" H 1000 2950 50  0001 C CNN
 F 1 "GND" H 1005 3027 50  0000 C CNN
 F 2 "" H 1000 3200 50  0001 C CNN
@@
 	3400 3200 3550 3200
 $Comp
-L power:GND #PWR?
+L power:GND #PWR0125
 U 1 1 5DE2363E
 P 3000 6350
-F 0 "#PWR?" H 3000 6100 50  0001 C CNN
+F 0 "#PWR0125" H 3000 6100 50  0001 C CNN
 F 1 "GND" H 3005 6177 50  0000 C CNN
 F 2 "" H 3000 6350 50  0001 C CNN
@@
 Connection ~ 2700 6200
 $Comp
-L power:GND #PWR?
+L power:GND #PWR0126
 U 1 1 5DE26E19
 P 1000 1500
-F 0 "#PWR?" H 1000 1250 50  0001 C CNN
+F 0 "#PWR0126" H 1000 1250 50  0001 C CNN
 F 1 "GND" H 1005 1327 50  0000 C CNN
 F 2 "" H 1000 1500 50  0001 C CNN
@@
 $EndComp
 $Comp
-L power:VDD #PWR?
+L power:VDD #PWR0127
 U 1 1 5DE28117
 P 1000 1100
-F 0 "#PWR?" H 1000 950 50  0001 C CNN
+F 0 "#PWR0127" H 1000 950 50  0001 C CNN
 F 1 "VDD" H 1017 1273 50  0000 C CNN
 F 2 "" H 1000 1100 50  0001 C CNN
@@
 $EndComp
 $Comp
-L Device:C_Small C?
+L Device:C_Small C3
 U 1 1 5DE28939
 P 1300 1300
-F 0 "C?" H 1392 1346 50  0000 L CNN
+F 0 "C3" H 1392 1346 50  0000 L CNN
 F 1 "10u" H 1392 1255 50  0000 L CNN
-F 2 "" H 1300 1300 50  0001 C CNN
+F 2 "Capacitor_SMD:C_0603_1608Metric_Pad1.05x0.95mm_HandSolder" H 1300 1300 50  0001 C CNN
 F 3 "~" H 1300 1300 50  0001 C CNN
 	1    1300 1300
@@
 $EndComp
 $Comp
-L Device:C_Small C?
+L Device:C_Small C4
 U 1 1 5DE28EDB
 P 1650 1300
-F 0 "C?" H 1742 1346 50  0000 L CNN
+F 0 "C4" H 1742 1346 50  0000 L CNN
 F 1 "100n" H 1742 1255 50  0000 L CNN
-F 2 "" H 1650 1300 50  0001 C CNN
+F 2 "Capacitor_SMD:C_0603_1608Metric_Pad1.05x0.95mm_HandSolder" H 1650 1300 50  0001 C CNN
 F 3 "~" H 1650 1300 50  0001 C CNN
 	1    1650 1300
@@
 	1300 1400 1650 1400
 $Comp
-L Device:C_Small C?
+L Device:C_Small C5
 U 1 1 5DE2D31C
 P 2100 1300
-F 0 "C?" H 2192 1346 50  0000 L CNN
+F 0 "C5" H 2192 1346 50  0000 L CNN
 F 1 "10u" H 2192 1255 50  0000 L CNN
-F 2 "" H 2100 1300 50  0001 C CNN
+F 2 "Capacitor_SMD:C_0603_1608Metric_Pad1.05x0.95mm_HandSolder" H 2100 1300 50  0001 C CNN
 F 3 "~" H 2100 1300 50  0001 C CNN
 	1    2100 1300
@@
 $EndComp
 $Comp
-L Device:C_Small C?
+L Device:C_Small C6
 U 1 1 5DE2D322
 P 2450 1300
-F 0 "C?" H 2542 1346 50  0000 L CNN
+F 0 "C6" H 2542 1346 50  0000 L CNN
 F 1 "100n" H 2542 1255 50  0000 L CNN
-F 2 "" H 2450 1300 50  0001 C CNN
+F 2 "Capacitor_SMD:C_0603_1608Metric_Pad1.05x0.95mm_HandSolder" H 2450 1300 50  0001 C CNN
 F 3 "~" H 2450 1300 50  0001 C CNN
 	1    2450 1300
@@
 	2100 1400 2450 1400
 $Comp
-L Device:C_Small C?
+L Device:C_Small C7
 U 1 1 5DE2EB1D
 P 2900 1300
-F 0 "C?" H 2992 1346 50  0000 L CNN
+F 0 "C7" H 2992 1346 50  0000 L CNN
 F 1 "10u" H 2992 1255 50  0000 L CNN
-F 2 "" H 2900 1300 50  0001 C CNN
+F 2 "Capacitor_SMD:C_0603_1608Metric_Pad1.05x0.95mm_HandSolder" H 2900 1300 50  0001 C CNN
 F 3 "~" H 2900 1300 50  0001 C CNN
 	1    2900 1300
@@
 $EndComp
 $Comp
-L Device:C_Small C?
+L Device:C_Small C8
 U 1 1 5DE2EB23
 P 3250 1300
-F 0 "C?" H 3342 1346 50  0000 L CNN
+F 0 "C8" H 3342 1346 50  0000 L CNN
 F 1 "100n" H 3342 1255 50  0000 L CNN
-F 2 "" H 3250 1300 50  0001 C CNN
+F 2 "Capacitor_SMD:C_0603_1608Metric_Pad1.05x0.95mm_HandSolder" H 3250 1300 50  0001 C CNN
 F 3 "~" H 3250 1300 50  0001 C CNN
 	1    3250 1300
@@
 	2900 1400 3250 1400
 $Comp
-L Device:C_Small C?
+L Device:C_Small C9
 U 1 1 5DE30029
 P 3650 1300
-F 0 "C?" H 3742 1346 50  0000 L CNN
+F 0 "C9" H 3742 1346 50  0000 L CNN
 F 1 "10u" H 3742 1255 50  0000 L CNN
-F 2 "" H 3650 1300 50  0001 C CNN
+F 2 "Capacitor_SMD:C_0603_1608Metric_Pad1.05x0.95mm_HandSolder" H 3650 1300 50  0001 C CNN
 F 3 "~" H 3650 1300 50  0001 C CNN
 	1    3650 1300
@@
 $EndComp
 $Comp
-L Device:C_Small C?
+L Device:C_Small C10
 U 1 1 5DE3002F
 P 4000 1300
-F 0 "C?" H 4092 1346 50  0000 L CNN
+F 0 "C10" H 4092 1346 50  0000 L CNN
 F 1 "100n" H 4092 1255 50  0000 L CNN
-F 2 "" H 4000 1300 50  0001 C CNN
+F 2 "Capacitor_SMD:C_0603_1608Metric_Pad1.05x0.95mm_HandSolder" H 4000 1300 50  0001 C CNN
 F 3 "~" H 4000 1300 50  0001 C CNN
 	1    4000 1300
@@
 	3550 3400 3400 3400
 $Comp
-L Device:C_Small C?
+L Device:C_Small C13
 U 1 1 5DE6A205
 P 1900 3200
-F 0 "C?" V 2129 3200 50  0000 C CNN
+F 0 "C13" V 2129 3200 50  0000 C CNN
 F 1 "4.7u" V 2038 3200 50  0000 C CNN
-F 2 "" H 1900 3200 50  0001 C CNN
+F 2 "Capacitor_SMD:C_0603_1608Metric_Pad1.05x0.95mm_HandSolder" H 1900 3200 50  0001 C CNN
 F 3 "~" H 1900 3200 50  0001 C CNN
 	1    1900 3200
@@
 SDA
 $Comp
-L Device:R_Small R?
+L Device:R_Small R11
 U 1 1 5DED1FCD
 P 3950 5400
-F 0 "R?" V 3754 5400 50  0000 C CNN
+F 0 "R11" V 3754 5400 50  0000 C CNN
 F 1 "4.7k" V 3845 5400 50  0000 C CNN
-F 2 "" H 3950 5400 50  0001 C CNN
+F 2 "Resistor_SMD:R_0603_1608Metric_Pad1.05x0.95mm_HandSolder" H 3950 5400 50  0001 C CNN
 F 3 "~" H 3950 5400 50  0001 C CNN
 	1    3950 5400
@@
 $EndComp
 $Comp
-L Device:R_Small R?
+L Device:R_Small R10
 U 1 1 5DED24A9
 P 3950 5100
-F 0 "R?" V 3754 5100 50  0000 C CNN
+F 0 "R10" V 3754 5100 50  0000 C CNN
 F 1 "4.7k" V 3845 5100 50  0000 C CNN
-F 2 "" H 3950 5100 50  0001 C CNN
+F 2 "Resistor_SMD:R_0603_1608Metric_Pad1.05x0.95mm_HandSolder" H 3950 5100 50  0001 C CNN
 F 3 "~" H 3950 5100 50  0001 C CNN
 	1    3950 5100
@@
 $EndComp
 $Comp
-L power:VDD #PWR?
+L power:VDD #PWR0128
 U 1 1 5DED283A
 P 4450 5100
-F 0 "#PWR?" H 4450 4950 50  0001 C CNN
+F 0 "#PWR0128" H 4450 4950 50  0001 C CNN
 F 1 "VDD" H 4467 5273 50  0000 C CNN
 F 2 "" H 4450 5100 50  0001 C CNN
@@
 	3550 5100 3850 5100
 $Comp
-L Device:R_Small R?
+L Device:R_Small R9
 U 1 1 5DEDFF14
 P 1300 3100
-F 0 "R?" V 1104 3100 50  0000 C CNN
+F 0 "R9" V 1104 3100 50  0000 C CNN
 F 1 "100k" V 1195 3100 50  0000 C CNN
-F 2 "" H 1300 3100 50  0001 C CNN
+F 2 "Resistor_SMD:R_0603_1608Metric_Pad1.05x0.95mm_HandSolder" H 1300 3100 50  0001 C CNN
 F 3 "~" H 1300 3100 50  0001 C CNN
 	1    1300 3100

Commit message: do initial layout
Connections:
- net CS2: now also U2.33 (PB12)
- net MISO2: now also U2.35 (PB14)
- net MOSI2: now also U2.36 (PB15)
- net SCK2: now also U2.34 (PB13)
Changed lines of the file:
@@
 Wire Wire Line
 	1200 3100 1200 3200
+Wire Wire Line
+	3400 5700 3550 5700
+Wire Wire Line
+	3400 5800 3550 5800
+Wire Wire Line
+	3550 5900 3400 5900
+Wire Wire Line
+	3400 6000 3550 6000
 $EndSCHEMATC
