File: blackbox-ng/blackbox-ng.sch (KiCad schematic (older format))
At the start: 24 parts, among them J1 CONN_DEBUG, J2 JST_PH, J3 CARD1, J4 CARD2, J5 Conn_01x08, J6 UART, SW1 SW_Push, SW2 SW_Push, U1 AP2112K-3.3

Commit message: do initial layout
Parts:
- J5: footprint Connector_PinHeader_2.54mm:PinHeader_1x08_P2.54mm_Vertical -> blackbox-ng:505110-0892
Connections:
- net at SW2.2: now also JP1.1
Changed lines of the file:
@@
 F 0 "J5" V 972 7980 50  0000 L CNN
 F 1 "Conn_01x08" V 1063 7980 50  0000 L CNN
-F 2 "Connector_PinHeader_2.54mm:PinHeader_1x08_P2.54mm_Vertical" H 1100 7600 50  0001 C CNN
+F 2 "blackbox-ng:505110-0892" H 1100 7600 50  0001 C CNN
 F 3 "~" H 1100 7600 50  0001 C CNN
 	1    1100 7600
@@
 Text Notes 9150 6950 2    200  ~ 0
 BLACKBOX V3
+Wire Wire Line
+	2900 6600 2850 6600
 $EndSCHEMATC
