File: blackbox-ng/blackbox-ng.kicad_pcb (KiCad board)
At the start: 2 copper layers, 48.3 x 43.2 mm, 52 parts, among them J1 CONN_DEBUG, J2 JST_PH, J3 CARD1, J4 CARD2, J5 Conn_01x08, J6 UART, SW1 SW_Push, SW2 SW_Push, U1 AP2112K-3.3, U2 STM32F401RETx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

Commit message: add very important board functionality
Parts:
- added G***: LOGO, FLOOF:husky-silk, F.Cu at (129.8, 106.7)
- added G***: LOGO, FLOOF:husky-mask, F.Cu at (129.8, 106.7)
- added G***: LOGO, FLOOF:husky-cu, F.Cu at (129.8, 106.7)
- added G***: LOGO, FLOOF:cat-face-trace, B.Cu at (134.4, 82.3)
- added G***: LOGO, FLOOF:cat-face-silk, B.Cu at (134.4, 82.3)
- added G***: LOGO, FLOOF:cat-face-gold, B.Cu at (134.4, 82.3)

Commit message: something something golden bears
Parts:
- added G***: LOGO, FLOOF:bear, F.Cu at (135.9, 78.0)

Commit message: cleanup layout
Parts:
- removed the G*** at (135.9, 78.0)
- added REF**: MountingHole_3mm_Pad, MountingHole:MountingHole_3mm_Pad, F.Cu at (171.4, 80.0)
- added REF**: MountingHole_3mm_Pad, MountingHole:MountingHole_3mm_Pad, F.Cu at (171.4, 115.6)
- added REF**: MountingHole_3mm_Pad, MountingHole:MountingHole_3mm_Pad, F.Cu at (131.1, 115.6)
- added REF**: MountingHole_3mm_Pad, MountingHole:MountingHole_3mm_Pad, F.Cu at (131.1, 80.0)
- moved G*** 26.7 mm to (131.6, 107.2)
- moved G*** 15.1 mm to (143.8, 112.5) (x3)
- moved R8 8.17 mm to (161.9, 80.8), turned to 180 degrees
- moved J6 7.88 mm to (165.7, 78.2)
- moved J1 6.08 mm to (173.1, 85.2)
- moved SW1 5.85 mm to (162.8, 114.0)
- moved R7 5.76 mm to (165.6, 82.3), turned to 180 degrees
- moved SW2 5.59 mm to (152.4, 114.0)
- moved TP1 5.50 mm to (157.7, 78.0)
- moved G*** 5.04 mm to (137.7, 86.1) (x3)
- moved J4 3.05 mm to (159.8, 108.5)
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Routing:
- net SCK1: track 42.4 -> 32.0 mm, vias 2 -> 1
- net NRST: track 73.3 -> 63.0 mm
- net VDD: track 214.1 -> 221.5 mm, vias 11 -> 13
- net RX: track 43.2 -> 49.3 mm
- net GND: track 93.2 -> 87.9 mm, vias 19 -> 20
- net MOSI1: track 32.3 -> 27.7 mm, vias 2 -> 1
- net Net-(JP1-Pad1): track 11.1 -> 15.3 mm
- net SDA: track 23.3 -> 27.2 mm
- net CS1-2: track 11.8 -> 15.2 mm
- net CS1-1: track 10.9 -> 8.13 mm
- net MISO1: track 34.5 -> 31.8 mm, vias 1 -> 3
- net SWO: track 16.5 -> 14.0 mm, vias 1 -> 0
- net TX: track 30.6 -> 32.8 mm
- net Net-(J6-Pad2): track 2.68 -> 4.70 mm
- net SCL: track 21.9 -> 23.8 mm
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
Commit message: fleshed out daughter card
Parts:
- removed REF** (x2): MountingHole_3mm_Pad, MountingHole:MountingHole_3mm_Pad
- added H2: MountingHole_3mm_Pad, MountingHole:MountingHole_3mm_Pad, F.Cu at (171.4, 80.0)
- added H3: MountingHole_3mm_Pad, MountingHole:MountingHole_3mm_Pad, F.Cu at (171.4, 115.6)
- renumbered REF** to H1, REF** to H4
Connections:
- H1 pad 1: (no net) -> GND
- H4 pad 1: (no net) -> GND
Routing:
- net GND: vias 20 -> 42
Changed lines of the file:
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@@
     (thickness 1.6)
     (drawings 11)
-    (tracks 577)
+    (tracks 599)
     (zones 0)
     (modules 62)
@@
   )
   (setup
-    (last_trace_width 0.254)
+    (last_trace_width 0.25)
     (user_trace_width 0.1524)
     (user_trace_width 0.254)
@@
     (mod_text_size 1 1)
     (mod_text_width 0.15)
-    (pad_size 1.524 1.524)
-    (pad_drill 0.762)
+    (pad_size 6.000001 6.000001)
+    (pad_drill 2.999999)
     (pad_to_mask_clearance 0.051)
     (solder_mask_min_width 0.25)
@@
     (pcbplotparams
       (layerselection 0x010fc_ffffffff)
-      (usegerberextensions false)
+      (usegerberextensions true)
       (usegerberattributes false)
       (usegerberadvancedattributes false)
@@
     (tags "mounting hole 3mm")
     (attr virtual)
-    (fp_text reference REF** (at -4.699 2.286) (layer B.SilkS)
-      (effects (font (size 1 1) (thickness 0.15)) (justify mirror))
+    (fp_text reference H2 (at -3.302 2.794) (layer F.SilkS)
+      (effects (font (size 1 1) (thickness 0.15)))
     )
     (fp_text value MountingHole_3mm_Pad (at 0 4) (layer F.Fab)
@@
     (fp_circle (center 0 0) (end 3 0) (layer Cmts.User) (width 0.15))
     (fp_circle (center 0 0) (end 3.25 0) (layer F.CrtYd) (width 0.05))
-    (pad 1 thru_hole circle (at 0 0) (size 6 6) (drill 3) (layers *.Cu *.Mask))
+    (pad 1 thru_hole circle (at 0 0) (size 6.000001 6.000001) (drill 2.999999) (layers *.Cu *.Mask)
+      (net 1 GND))
   )
   (module MountingHole:MountingHole_3mm_Pad (layer F.Cu)
@@
     (tags "mounting hole 3mm")
     (attr virtual)
-    (fp_text reference REF** (at 0 -4.064) (layer F.SilkS)
+    (fp_text reference H3 (at 0 -4.064) (layer F.SilkS)
       (effects (font (size 1 1) (thickness 0.15)))
     )
@@
     (fp_circle (center 0 0) (end 3 0) (layer Cmts.User) (width 0.15))
     (fp_circle (center 0 0) (end 3.25 0) (layer F.CrtYd) (width 0.05))
-    (pad 1 thru_hole circle (at 0 0) (size 6 6) (drill 3) (layers *.Cu *.Mask))
+    (pad 1 thru_hole circle (at 0 0) (size 6.000001 6.000001) (drill 2.999999) (layers *.Cu *.Mask)
+      (net 1 GND))
   )
   (module blehhhh:MOLEX_500901-0801 (layer B.Cu)
@@
     (tags "mounting hole 3mm")
     (attr virtual)
-    (fp_text reference REF** (at 0 -4) (layer F.SilkS)
+    (fp_text reference H4 (at 0 -4) (layer F.SilkS)
       (effects (font (size 1 1) (thickness 0.15)))
     )
@@
       (effects (font (size 1 1) (thickness 0.15)))
     )
-    (pad 1 thru_hole circle (at 0 0) (size 6 6) (drill 3) (layers *.Cu *.Mask))
+    (pad 1 thru_hole circle (at 0 0) (size 6.000001 6.000001) (drill 2.999999) (layers *.Cu *.Mask)
+      (net 1 GND))
   )
   (module MountingHole:MountingHole_3mm_Pad (layer F.Cu)
@@
     (tags "mounting hole 3mm")
     (attr virtual)
-    (fp_text reference REF** (at 0.127 3.937) (layer F.SilkS)
+    (fp_text reference H1 (at 0 4.064) (layer F.SilkS)
       (effects (font (size 1 1) (thickness 0.15)))
     )
@@
       (effects (font (size 1 1) (thickness 0.15)))
     )
-    (pad 1 thru_hole circle (at 0 0) (size 6 6) (drill 3) (layers *.Cu *.Mask))
+    (pad 1 thru_hole circle (at 0 0) (size 6.000001 6.000001) (drill 2.999999) (layers *.Cu *.Mask)
+      (net 1 GND))
   )
   (module FLOOF:star (layer F.Cu)
@@
   (segment (start 171.45 88.392) (end 165.6585 88.392) (width 0.254) (layer B.Cu) (net 1))
   (via (at 165.0235 87.757) (size 0.8) (drill 0.4) (layers F.Cu B.Cu) (net 1))
+  (via (at 139.954 115.57) (size 0.8) (drill 0.4) (layers F.Cu B.Cu) (net 1))
+  (via (at 143.51 117.094) (size 0.8) (drill 0.4) (layers F.Cu B.Cu) (net 1))
+  (via (at 162.56 114.046) (size 0.8) (drill 0.4) (layers F.Cu B.Cu) (net 1))
+  (via (at 159.004 114.3) (size 0.8) (drill 0.4) (layers F.Cu B.Cu) (net 1))
+  (via (at 164.084 117.348) (size 0.8) (drill 0.4) (layers F.Cu B.Cu) (net 1))
+  (via (at 169.164 111.506) (size 0.8) (drill 0.4) (layers F.Cu B.Cu) (net 1))
+  (via (at 169.672 104.394) (size 0.8) (drill 0.4) (layers F.Cu B.Cu) (net 1))
+  (via (at 158.496 101.092) (size 0.8) (drill 0.4) (layers F.Cu B.Cu) (net 1))
+  (via (at 160.528 96.266) (size 0.8) (drill 0.4) (layers F.Cu B.Cu) (net 1))
+  (via (at 164.846 94.996) (size 0.8) (drill 0.4) (layers F.Cu B.Cu) (net 1))
+  (via (at 135.128 95.25) (size 0.8) (drill 0.4) (layers F.Cu B.Cu) (net 1))
+  (via (at 134.366 101.346) (size 0.8) (drill 0.4) (layers F.Cu B.Cu) (net 1))
+  (via (at 132.08 102.616) (size 0.8) (drill 0.4) (layers F.Cu B.Cu) (net 1))
+  (via (at 128.524 111.252) (size 0.8) (drill 0.4) (layers F.Cu B.Cu) (net 1))
+  (via (at 133.858 112.014) (size 0.8) (drill 0.4) (layers F.Cu B.Cu) (net 1))
+  (via (at 137.668 117.348) (size 0.8) (drill 0.4) (layers F.Cu B.Cu) (net 1))
+  (via (at 136.906 108.204) (size 0.8) (drill 0.4) (layers F.Cu B.Cu) (net 1))
+  (via (at 143.002 101.092) (size 0.8) (drill 0.4) (layers F.Cu B.Cu) (net 1))
+  (via (at 148.082 97.282) (size 0.8) (drill 0.4) (layers F.Cu B.Cu) (net 1))
+  (via (at 149.86 99.314) (size 0.8) (drill 0.4) (layers F.Cu B.Cu) (net 1))
+  (via (at 143.002 91.186) (size 0.8) (drill 0.4) (layers F.Cu B.Cu) (net 1))
+  (via (at 149.86 84.074) (size 0.8) (drill 0.4) (layers F.Cu B.Cu) (net 1))
   (segment (start 147.941 98.806) (end 147.941 100.457) (width 0.2032) (layer B.Cu) (net 2))
   (via (at 147.941 100.457) (size 0.8) (drill 0.4) (layers F.Cu B.Cu) (net 2))

Commit message: made suggested edits
Parts:
- moved H1 0.25 mm to (130.8, 80.0)
- moved H4 0.25 mm to (130.8, 115.6)
Routing:
- net VDD: track 221.5 -> 223.2 mm
- net RX: track 49.3 -> 50.6 mm
- net SDA: track 27.2 -> 26.2 mm
- net CS1-2: track 15.2 -> 15.7 mm
- net GND: vias 42 -> 56
Other:
- outline, holes or cut-outs redrawn
